File: 555 timer.sch (KiCad schematic (older format))
At the start: 3 parts

Commit message: created pcb
Parts:
- R10: renamed from R?; footprint Kicad_lib:R_0603 -> MAIN_PCB_LIB:R_0603
- gave numbers to parts that had none: 2
Changed lines of the file:
@@
 $Descr A4 11693 8268
 encoding utf-8
-Sheet 4 4
+Sheet 4 5
 Title ""
 Date ""
@@
 $EndDescr
 $Comp
-L Main_Library:U_555_timer U?
+L Main_Library:U_555_timer U6
 U 1 1 6158C04F
 P 5900 2900
-F 0 "U?" H 5900 2577 50  0000 C CNN
+F 0 "U6" H 5900 2577 50  0000 C CNN
 F 1 "U_555_timer" H 5900 2486 50  0000 C CNN
 F 2 "MAIN_PCB_LIB:U_LM555CN" H 5900 3400 50  0001 C CNN
@@
 Connection ~ 6050 2550
 $Comp
-L Main_Library:GND #GND?
+L Main_Library:GND #GND021
 U 1 1 6158C8C7
 P 5600 2450
-F 0 "#GND?" H 5440 2430 50  0001 C CNN
+F 0 "#GND021" H 5440 2430 50  0001 C CNN
 F 1 "GND" H 5440 2430 50  0001 C CNN
 F 2 "" H 5510 2390 50  0001 C CNN
@@
 	5800 2450 5600 2450
 $Comp
-L Main_Library:R_2K_0603 R?
+L Main_Library:R_2K_0603 R10
 U 1 1 6158D370
 P 6450 2900
-F 0 "R?" V 6260 2900 50  0000 C CNN
+F 0 "R10" V 6260 2900 50  0000 C CNN
 F 1 "R_2K_0603" H 6800 3000 50  0001 C CNN
-F 2 "Kicad_lib:R_0603" H 6500 3400 50  0001 C CNN
+F 2 "MAIN_PCB_LIB:R_0603" H 6500 3400 50  0001 C CNN
 F 3 "" H 6450 3150 50  0001 C CNN
 F 4 "603-RT0603BRD072KL" H 6450 3400 50  0001 C CNN "Mouser"
@@
 Connection ~ 5550 2900
 $Comp
-L Main_Library:C_1nF_0603_50V C?
+L Main_Library:C_1nF_0603_50V C8
 U 1 1 61590D9D
 P 5250 3050
-F 0 "C?" H 5328 3096 50  0000 L CNN
+F 0 "C8" H 5328 3096 50  0000 L CNN
 F 1 "C_1nF_0603_50V" H 5300 3400 50  0001 C CNN
 F 2 "MAIN_PCB_LIB:C_0603" H 5300 3400 50  0001 C CNN
@@
 $EndComp
 $Comp
-L Main_Library:GND #GND?
+L Main_Library:GND #GND020
 U 1 1 61591AE3
 P 5250 3200
-F 0 "#GND?" H 5090 3180 50  0001 C CNN
+F 0 "#GND020" H 5090 3180 50  0001 C CNN
 F 1 "GND" H 5090 3180 50  0001 C CNN
 F 2 "" H 5160 3140 50  0001 C CNN
