File: VU-Meter.sch (KiCad schematic (older format))
At the start: 15 parts, among them U7 U_LM3914N-1_NOPB

Commit message: changed vu meter resistor value's
Parts:
- removed R13: R_3K4_0603, MAIN_PCB_LIB:R_0603, symbol Main_Library:R_3K4_0603
- R11: Waarde 4K7 -> 91K
- R12: Waarde 1K -> 18K
Connections:
- wire segments 56 -> 53
Other:
- moved on the sheet: R14
Changed lines of the file:
@@
 EESchema Schematic File Version 4
-LIBS:versterker-cache
 EELAYER 30 0
 EELAYER END
@@
 F 2 "MAIN_PCB_LIB:R_0603" H 5000 4270 50  0001 C CNN
 F 3 "" H 4750 3600 50  0001 C CNN
-F 4 "1K" H 4852 3705 50  0000 L CNN "Waarde"
+F 4 "18K" H 4852 3705 50  0000 L CNN "Waarde"
 F 5 "311-1.0KDDKR-ND" H 4950 4350 50  0001 C CNN "Digi-Key"
 	1    4800 3750
@@
 F 2 "MAIN_PCB_LIB:R_0603" H 4600 3700 50  0001 C CNN
 F 3 "" H 4600 3700 50  0001 C CNN
-F 4 "4K7" V 4700 3550 50  0000 C CNN "Waarde"
+F 4 "91K" V 4700 3550 50  0000 C CNN "Waarde"
 	1    4600 3550
 	0    1    1    0
@@
 L Main_Library:R_3K16_0603 R14
 U 1 1 61702C03
-P 5350 4350
-F 0 "R14" V 5252 4350 50  0000 C CNN
-F 1 "R_3K16_0603" H 5350 4350 50  0001 C CNN
-F 2 "MAIN_PCB_LIB:R_0603" H 5350 4350 50  0001 C CNN
-F 3 "" H 5350 4350 50  0001 C CNN
-F 4 "603-RT0603BRD073K16L" H 5350 4350 50  0001 C CNN "mouser"
-F 5 "3K16" V 5400 4350 50  0000 C CNN "Waarde"
-	1    5350 4350
-	0    1    1    0
-$EndComp
-$Comp
-L Main_Library:R_3K4_0603 R13
-U 1 1 616F387C
-P 4950 4350
-F 0 "R13" V 5003 4388 39  0000 L CNN
-F 1 "R_3K4_0603" H 4850 4750 39  0001 C CNN
-F 2 "MAIN_PCB_LIB:R_0603" H 4850 4800 39  0001 C CNN
-F 3 "" H 4850 4450 39  0001 C CNN
-F 4 "3K4" V 4900 4300 39  0000 L CNN "Waarde"
-F 5 "667-ERJ-3EKF3401V" H 4800 4850 39  0001 C CNN "Mouser"
-	1    4950 4350
-	0    -1   -1   0
-$EndComp
-Wire Wire Line
-	5550 4350 5800 4350
+P 5800 4550
+F 0 "R14" V 5702 4550 50  0000 C CNN
+F 1 "R_3K16_0603" H 5800 4550 50  0001 C CNN
+F 2 "MAIN_PCB_LIB:R_0603" H 5800 4550 50  0001 C CNN
+F 3 "" H 5800 4550 50  0001 C CNN
+F 4 "603-RT0603BRD073K16L" H 5800 4550 50  0001 C CNN "mouser"
+F 5 "3K16" V 5850 4550 50  0000 C CNN "Waarde"
+	1    5800 4550
+	1    0    0    -1
+$EndComp
 Wire Wire Line
 	5800 4350 5800 4050
@@
 Wire Wire Line
 	5800 4350 5850 4350
-$Comp
-L Main_Library:GND #GND022
-U 1 1 616F7F03
-P 4750 4350
-F 0 "#GND022" H 4590 4330 50  0001 C CNN
-F 1 "GND" H 4590 4330 50  0001 C CNN
-F 2 "" H 4660 4290 50  0001 C CNN
-F 3 "" H 4660 4290 50  0001 C CNN
-	1    4750 4350
-	1    0    0    -1
-$EndComp
-Wire Wire Line
-	5150 4350 5150 4250
-Wire Wire Line
-	5150 4250 5850 4250
-Connection ~ 5150 4350
-Wire Wire Line
-	5150 4250 5150 3950
-Connection ~ 5150 4250
-Wire Wire Line
-	5150 3950 5850 3950
 Wire Wire Line
 	4800 3550 5850 3550
@@
 Wire Wire Line
 	8700 3300 8700 3000
+$Comp
+L Main_Library:GND #GND?
+U 1 1 619BE6AF
+P 5650 3950
+F 0 "#GND?" H 5490 3930 50  0001 C CNN
+F 1 "GND" H 5490 3930 50  0001 C CNN
+F 2 "" H 5560 3890 50  0001 C CNN
+F 3 "" H 5560 3890 50  0001 C CNN
+	1    5650 3950
+	1    0    0    -1
+$EndComp
+Wire Wire Line
+	5850 3950 5650 3950
+$Comp
+L Main_Library:GND #GND?
+U 1 1 619C0A27
+P 5800 4750
+F 0 "#GND?" H 5640 4730 50  0001 C CNN
+F 1 "GND" H 5640 4730 50  0001 C CNN
+F 2 "" H 5710 4690 50  0001 C CNN
+F 3 "" H 5710 4690 50  0001 C CNN
+	1    5800 4750
+	1    0    0    -1
+$EndComp
+$Comp
+L Main_Library:GND #GND?
+U 1 1 619C1A09
+P 5600 4250
+F 0 "#GND?" H 5440 4230 50  0001 C CNN
+F 1 "GND" H 5440 4230 50  0001 C CNN
+F 2 "" H 5510 4190 50  0001 C CNN
+F 3 "" H 5510 4190 50  0001 C CNN
+	1    5600 4250
+	1    0    0    -1
+$EndComp
+Wire Wire Line
+	5850 4250 5600 4250
 $EndSCHEMATC

Commit message: added raspberry pi hat pcb outline and layout
Parts:
- renumbered R11 to R16, R12 to R17, R14 to R18, U7 to U6
Changed lines of the file:
@@
 Signal
 $Comp
-L Main_Library:U_LM3914N-1_NOPB U7
+L Main_Library:U_LM3914N-1_NOPB U6
 U 1 1 616F242F
 P 5750 3350
-F 0 "U7" H 6550 3523 50  0000 C CNN
+F 0 "U6" H 6550 3523 50  0000 C CNN
 F 1 "U_LM3914N-1_NOPB" H 5750 3650 50  0001 L CNN
 F 2 "MAIN_PCB_LIB:U_LM3914_TI_DIP" H 5750 3750 50  0001 L CNN
@@
 $EndComp
 $Comp
-L Main_Library:R_1K_0603 R12
+L Main_Library:R_1K_0603 R17
 U 1 1 616F5590
 P 4800 3750
-F 0 "R12" H 4852 3796 50  0000 L CNN
+F 0 "R17" H 4852 3796 50  0000 L CNN
 F 1 "R_1K_0603" H 4800 4200 50  0001 C CNN
 F 2 "MAIN_PCB_LIB:R_0603" H 5000 4270 50  0001 C CNN
@@
 $EndComp
 $Comp
-L Main_Library:GND #GND023
+L Main_Library:GND #GND020
 U 1 1 616F61AA
 P 4800 3950
-F 0 "#GND023" H 4640 3930 50  0001 C CNN
+F 0 "#GND020" H 4640 3930 50  0001 C CNN
 F 1 "GND" H 4640 3930 50  0001 C CNN
 F 2 "" H 4710 3890 50  0001 C CNN
@@
 $EndComp
 $Comp
-L Main_Library:R_4K7_0603 R11
+L Main_Library:R_4K7_0603 R16
 U 1 1 616FA265
 P 4600 3550
-F 0 "R11" V 4550 3550 50  0000 C CNN
+F 0 "R16" V 4550 3550 50  0000 C CNN
 F 1 "R_4K7_0603" V 4375 3550 50  0001 C CNN
 F 2 "MAIN_PCB_LIB:R_0603" H 4600 3700 50  0001 C CNN
@@
 Connection ~ 4800 3550
 $Comp
-L Main_Library:R_3K16_0603 R14
+L Main_Library:R_3K16_0603 R18
 U 1 1 61702C03
 P 5800 4550
-F 0 "R14" V 5702 4550 50  0000 C CNN
+F 0 "R18" V 5702 4550 50  0000 C CNN
 F 1 "R_3K16_0603" H 5800 4550 50  0001 C CNN
 F 2 "MAIN_PCB_LIB:R_0603" H 5800 4550 50  0001 C CNN
@@
 	8700 3300 8700 3000
 $Comp
-L Main_Library:GND #GND?
+L Main_Library:GND #GND022
 U 1 1 619BE6AF
 P 5650 3950
-F 0 "#GND?" H 5490 3930 50  0001 C CNN
+F 0 "#GND022" H 5490 3930 50  0001 C CNN
 F 1 "GND" H 5490 3930 50  0001 C CNN
 F 2 "" H 5560 3890 50  0001 C CNN
@@
 	5850 3950 5650 3950
 $Comp
-L Main_Library:GND #GND?
+L Main_Library:GND #GND023
 U 1 1 619C0A27
 P 5800 4750
-F 0 "#GND?" H 5640 4730 50  0001 C CNN
+F 0 "#GND023" H 5640 4730 50  0001 C CNN
 F 1 "GND" H 5640 4730 50  0001 C CNN
 F 2 "" H 5710 4690 50  0001 C CNN
@@
 $EndComp
 $Comp
-L Main_Library:GND #GND?
+L Main_Library:GND #GND021
 U 1 1 619C1A09
 P 5600 4250
-F 0 "#GND?" H 5440 4230 50  0001 C CNN
+F 0 "#GND021" H 5440 4230 50  0001 C CNN
 F 1 "GND" H 5440 4230 50  0001 C CNN
 F 2 "" H 5510 4190 50  0001 C CNN

Commit message: changed vu meter circuit
Parts:
- removed R16: R_4K7_0603, MAIN_PCB_LIB:R_0603, symbol Main_Library:R_4K7_0603
- removed R17: R_1K_0603, MAIN_PCB_LIB:R_0603, symbol Main_Library:R_1K_0603
- added C1: C_10uF_0603, MAIN_PCB_LIB:C_0603, symbol Main_Library:C_10uF_0603
- added D13, D14: D_1N4148WS_SOD323F_ONSEMI, MAIN_PCB_LIB:D_1N4148_SOD-323F_ONSEMI, symbol Main_Library:D_1N4148WS_SOD323F_ONSEMI
- added R16: R_25K5_0603, MAIN_PCB_LIB:R_0603, symbol Main_Library:R_25K5_0603
- added R17, R2: R_10K_0603, MAIN_PCB_LIB:R_0603, symbol Main_Library:R_10K_0603
- added R3: R_2K_0603, MAIN_PCB_LIB:R_0603, symbol Main_Library:R_2K_0603
Other:
- note added: "1.5v"
- note added: "3.6v"
- moved on the sheet: R18
Changed lines of the file:
@@
 $Descr A4 11693 8268
 encoding utf-8
-Sheet 5 4
+Sheet 4 4
 Title ""
 Date ""
@@
 Comment4 ""
 $EndDescr
-Text HLabel 4400 3350 0    50   Input ~ 0
+Text HLabel 5750 3350 0    50   Input ~ 0
 9V
-Text HLabel 4400 3550 0    50   Input ~ 0
+Text HLabel 4200 3550 0    50   Input ~ 0
 Signal
 $Comp
@@
 $EndComp
 $Comp
-L Main_Library:R_1K_0603 R17
-U 1 1 616F5590
-P 4800 3750
-F 0 "R17" H 4852 3796 50  0000 L CNN
-F 1 "R_1K_0603" H 4800 4200 50  0001 C CNN
-F 2 "MAIN_PCB_LIB:R_0603" H 5000 4270 50  0001 C CNN
-F 3 "" H 4750 3600 50  0001 C CNN
-F 4 "18K" H 4852 3705 50  0000 L CNN "Waarde"
-F 5 "311-1.0KDDKR-ND" H 4950 4350 50  0001 C CNN "Digi-Key"
-	1    4800 3750
-	1    0    0    -1
-$EndComp
-$Comp
-L Main_Library:GND #GND020
-U 1 1 616F61AA
-P 4800 3950
-F 0 "#GND020" H 4640 3930 50  0001 C CNN
-F 1 "GND" H 4640 3930 50  0001 C CNN
-F 2 "" H 4710 3890 50  0001 C CNN
-F 3 "" H 4710 3890 50  0001 C CNN
-	1    4800 3950
-	1    0    0    -1
-$EndComp
-$Comp
-L Main_Library:R_4K7_0603 R16
-U 1 1 616FA265
-P 4600 3550
-F 0 "R16" V 4550 3550 50  0000 C CNN
-F 1 "R_4K7_0603" V 4375 3550 50  0001 C CNN
-F 2 "MAIN_PCB_LIB:R_0603" H 4600 3700 50  0001 C CNN
-F 3 "" H 4600 3700 50  0001 C CNN
-F 4 "91K" V 4700 3550 50  0000 C CNN "Waarde"
-	1    4600 3550
-	0    1    1    0
-$EndComp
-Connection ~ 4800 3550
-$Comp
 L Main_Library:R_3K16_0603 R18
 U 1 1 61702C03
-P 5800 4550
-F 0 "R18" V 5702 4550 50  0000 C CNN
-F 1 "R_3K16_0603" H 5800 4550 50  0001 C CNN
-F 2 "MAIN_PCB_LIB:R_0603" H 5800 4550 50  0001 C CNN
-F 3 "" H 5800 4550 50  0001 C CNN
-F 4 "603-RT0603BRD073K16L" H 5800 4550 50  0001 C CNN "mouser"
-F 5 "3K16" V 5850 4550 50  0000 C CNN "Waarde"
-	1    5800 4550
-	1    0    0    -1
-$EndComp
-Wire Wire Line
-	5800 4350 5800 4050
-Wire Wire Line
-	5800 4050 5850 4050
-Connection ~ 5800 4350
-Wire Wire Line
-	5800 4350 5850 4350
-Wire Wire Line
-	4800 3550 5850 3550
-Wire Wire Line
-	4400 3350 5850 3350
-Text Label 4400 3350 0    50   ~ 0
+P 5650 4050
+F 0 "R18" V 5552 4050 50  0000 C CNN
+F 1 "R_3K16_0603" H 5650 4050 50  0001 C CNN
+F 2 "MAIN_PCB_LIB:R_0603" H 5650 4050 50  0001 C CNN
+F 3 "" H 5650 4050 50  0001 C CNN
+F 4 "603-RT0603BRD073K16L" H 5650 4050 50  0001 C CNN "mouser"
+F 5 "3K16" V 5700 4050 50  0000 C CNN "Waarde"
+	1    5650 4050
+	0    -1   -1   0
+$EndComp
+Text Label 5750 3350 0    50   ~ 0
 9V
 Text Label 5700 3750 0    50   ~ 0
@@
 L Main_Library:GND #GND022
 U 1 1 619BE6AF
-P 5650 3950
-F 0 "#GND022" H 5490 3930 50  0001 C CNN
-F 1 "GND" H 5490 3930 50  0001 C CNN
-F 2 "" H 5560 3890 50  0001 C CNN
-F 3 "" H 5560 3890 50  0001 C CNN
-	1    5650 3950
-	1    0    0    -1
-$EndComp
-Wire Wire Line
-	5850 3950 5650 3950
+P 5100 3950
+F 0 "#GND022" H 4940 3930 50  0001 C CNN
+F 1 "GND" H 4940 3930 50  0001 C CNN
+F 2 "" H 5010 3890 50  0001 C CNN
+F 3 "" H 5010 3890 50  0001 C CNN
+	1    5100 3950
+	1    0    0    -1
+$EndComp
 $Comp
 L Main_Library:GND #GND023
 U 1 1 619C0A27
-P 5800 4750
-F 0 "#GND023" H 5640 4730 50  0001 C CNN
-F 1 "GND" H 5640 4730 50  0001 C CNN
-F 2 "" H 5710 4690 50  0001 C CNN
-F 3 "" H 5710 4690 50  0001 C CNN
-	1    5800 4750
+P 5450 4050
+F 0 "#GND023" H 5290 4030 50  0001 C CNN
+F 1 "GND" H 5290 4030 50  0001 C CNN
+F 2 "" H 5360 3990 50  0001 C CNN
+F 3 "" H 5360 3990 50  0001 C CNN
+	1    5450 4050
+	1    0    0    -1
+$EndComp
+Wire Wire Line
+	5100 3950 5850 3950
+Wire Wire Line
+	5850 4250 5150 4250
+Text Label 4850 4250 2    50   ~ 0
+9V
+$Comp
+L Main_Library:R_10K_0603 R2
+U 1 1 61B47D7E
+P 5000 4250
+F 0 "R2" V 4834 4250 39  0000 C CNN
+F 1 "R_10K_0603" H 4950 4800 39  0001 C CNN
+F 2 "MAIN_PCB_LIB:R_0603" H 5000 4750 39  0001 C CNN
+F 3 "" H 4950 4400 39  0001 C CNN
+F 4 "10K" V 4909 4250 39  0000 C CNN "Waarde"
+F 5 "YAG1236CT-ND" H 5000 4850 39  0001 C CNN "Digi-key"
+	1    5000 4250
+	0    1    1    0
+$EndComp
+$Comp
+L Main_Library:R_2K_0603 R3
+U 1 1 61B509CE
+P 5150 4450
+F 0 "R3" H 5203 4496 50  0000 L CNN
+F 1 "R_2K_0603" H 5500 4550 50  0001 C CNN
+F 2 "MAIN_PCB_LIB:R_0603" H 5200 4950 50  0001 C CNN
+F 3 "" H 5150 4700 50  0001 C CNN
+F 4 "603-RT0603BRD072KL" H 5150 4950 50  0001 C CNN "Mouser"
+F 5 "2K" H 5203 4405 50  0000 L CNN "Waarde"
+	1    5150 4450
+	1    0    0    -1
+$EndComp
+Connection ~ 5150 4250
+$Comp
+L Main_Library:GND #GND05
+U 1 1 61B51C86
+P 5150 4650
+F 0 "#GND05" H 4990 4630 50  0001 C CNN
+F 1 "GND" H 4990 4630 50  0001 C CNN
+F 2 "" H 5060 4590 50  0001 C CNN
+F 3 "" H 5060 4590 50  0001 C CNN
+	1    5150 4650
+	1    0    0    -1
+$EndComp
+Text Notes 5150 4250 0    50   ~ 0
+1.5v
+$Comp
+L Main_Library:R_25K5_0603 R16
+U 1 1 61B5A423
+P 5550 4350
+F 0 "R16" V 5500 4350 50  0000 C CNN
+F 1 "R_25K5_0603" H 5550 4800 50  0001 C CNN
+F 2 "MAIN_PCB_LIB:R_0603" H 5750 4870 50  0001 C CNN
+F 3 "" H 5500 4200 50  0001 C CNN
+F 4 "25K5" V 5650 4350 50  0000 C CNN "Waarde"
+F 5 "603-RT0603FRE0725K5L" H 5700 4950 50  0001 C CNN "Digi-Key"
+	1    5550 4350
+	0    1    1    0
+$EndComp
+Text Label 5350 4350 2    50   ~ 0
+9V
+Wire Wire Line
+	5750 4350 5850 4350
+Text Notes 5750 4350 0    50   ~ 0
+3.6v
+Wire Wire Line
+	5750 3350 5850 3350
+$Comp
+L Main_Library:D_1N4148WS_SOD323F_ONSEMI D13
+U 1 1 61BAA2D9
+P 4400 3700
+F 0 "D13" V 4400 3778 50  0000 L CNN
+F 1 "D_1N4148WS_SOD323F_ONSEMI" H 4400 4100 50  0001 C CNN
+F 2 "MAIN_PCB_LIB:D_1N4148_SOD-323F_ONSEMI" H 4400 4000 50  0001 C CNN
+F 3 "" H 4400 4000 50  0001 C CNN
+F 4 "512-1N4148WS" H 4400 4250 50  0001 C CNN "Mouser"
+	1    4400 3700
+	0    1    1    0
+$EndComp
+$Comp
+L Main_Library:D_1N4148WS_SOD323F_ONSEMI D14
+U 1 1 61BAB237
+P 4550 3550
+F 0 "D14" H 4550 3427 50  0000 C CNN
+F 1 "D_1N4148WS_SOD323F_ONSEMI" H 4550 3950 50  0001 C CNN
+F 2 "MAIN_PCB_LIB:D_1N4148_SOD-323F_ONSEMI" H 4550 3850 50  0001 C CNN
+F 3 "" H 4550 3850 50  0001 C CNN
+F 4 "512-1N4148WS" H 4550 4100 50  0001 C CNN "Mouser"
+	1    4550 3550
+	-1   0    0    1
+$EndComp
+Wire Wire Line
+	4400 3550 4200 3550
+Connection ~ 4400 3550
+$Comp
+L Main_Library:GND #GND020
+U 1 1 61BADC2D
+P 4400 3850
+F 0 "#GND020" H 4240 3830 50  0001 C CNN
+F 1 "GND" H 4240 3830 50  0001 C CNN
+F 2 "" H 4310 3790 50  0001 C CNN
+F 3 "" H 4310 3790 50  0001 C CNN
+	1    4400 3850
+	1    0    0    -1
+$EndComp
+$Comp
+L Main_Library:C_10uF_0603 C1
+U 1 1 61BAF616
+P 4700 3700
+F 0 "C1" H 4778 3746 50  0000 L CNN
+F 1 "C_10uF_0603" H 4700 3950 50  0001 C CNN
+F 2 "MAIN_PCB_LIB:C_0603" H 4860 4020 50  0001 C CNN
+F 3 "" H 4640 3600 50  0001 C CNN
+F 4 "10uF" H 4778 3655 50  0000 L CNN "Waarde"
+F 5 "311-1448-2-ND" H 4700 3700 50  0001 C CNN "Digi-Key"
+	1    4700 3700
+	1    0    0    -1
+$EndComp
+$Comp
+L Main_Library:R_10K_0603 R17
+U 1 1 61BB845F
+P 5000 3700
+F 0 "R17" H 5100 3750 39  0000 C CNN
+F 1 "R_10K_0603" H 4950 4250 39  0001 C CNN
+F 2 "MAIN_PCB_LIB:R_0603" H 5000 4200 39  0001 C CNN
+F 3 "" H 4950 3850 39  0001 C CNN
+F 4 "10K" H 5100 3700 39  0000 C CNN "Waarde"
+F 5 "YAG1236CT-ND" H 5000 4300 39  0001 C CNN "Digi-key"
+	1    5000 3700
 	1    0    0    -1
 $EndComp
 $Comp
 L Main_Library:GND #GND021
-U 1 1 619C1A09
-P 5600 4250
-F 0 "#GND021" H 5440 4230 50  0001 C CNN
-F 1 "GND" H 5440 4230 50  0001 C CNN
-F 2 "" H 5510 4190 50  0001 C CNN
-F 3 "" H 5510 4190 50  0001 C CNN
-	1    5600 4250
-	1    0    0    -1
-$EndComp
-Wire Wire Line
-	5850 4250 5600 4250
+U 1 1 61BB9DB3
+P 4700 3850
+F 0 "#GND021" H 4540 3830 50  0001 C CNN
+F 1 "GND" H 4540 3830 50  0001 C CNN
+F 2 "" H 4610 3790 50  0001 C CNN
+F 3 "" H 4610 3790 50  0001 C CNN
+	1    4700 3850
+	1    0    0    -1
+$EndComp
+$Comp
+L Main_Library:GND #GND025
+U 1 1 61BBAE7D
+P 5000 3850
+F 0 "#GND025" H 4840 3830 50  0001 C CNN
+F 1 "GND" H 4840 3830 50  0001 C CNN
+F 2 "" H 4910 3790 50  0001 C CNN
+F 3 "" H 4910 3790 50  0001 C CNN
+	1    5000 3850
+	1    0    0    -1
+$EndComp
+Wire Wire Line
+	4700 3550 5000 3550
+Connection ~ 4700 3550
+Wire Wire Line
+	5000 3550 5850 3550
+Connection ~ 5000 3550
 $EndSCHEMATC

Commit message: routed pcb
Parts:
- removed R2: R_10K_0603, MAIN_PCB_LIB:R_0603, symbol Main_Library:R_10K_0603
- removed R3: R_2K_0603, MAIN_PCB_LIB:R_0603, symbol Main_Library:R_2K_0603
Other:
- note removed: "1.5v"
Changed lines of the file:
@@
 L Main_Library:GND #GND022
 U 1 1 619BE6AF
-P 5100 3950
-F 0 "#GND022" H 4940 3930 50  0001 C CNN
-F 1 "GND" H 4940 3930 50  0001 C CNN
-F 2 "" H 5010 3890 50  0001 C CNN
-F 3 "" H 5010 3890 50  0001 C CNN
-	1    5100 3950
+P 5350 3950
+F 0 "#GND022" H 5190 3930 50  0001 C CNN
+F 1 "GND" H 5190 3930 50  0001 C CNN
+F 2 "" H 5260 3890 50  0001 C CNN
+F 3 "" H 5260 3890 50  0001 C CNN
+	1    5350 3950
 	1    0    0    -1
 $EndComp
@@
 	1    0    0    -1
 $EndComp
-Wire Wire Line
-	5100 3950 5850 3950
-Wire Wire Line
-	5850 4250 5150 4250
-Text Label 4850 4250 2    50   ~ 0
-9V
-$Comp
-L Main_Library:R_10K_0603 R2
-U 1 1 61B47D7E
-P 5000 4250
-F 0 "R2" V 4834 4250 39  0000 C CNN
-F 1 "R_10K_0603" H 4950 4800 39  0001 C CNN
-F 2 "MAIN_PCB_LIB:R_0603" H 5000 4750 39  0001 C CNN
-F 3 "" H 4950 4400 39  0001 C CNN
-F 4 "10K" V 4909 4250 39  0000 C CNN "Waarde"
-F 5 "YAG1236CT-ND" H 5000 4850 39  0001 C CNN "Digi-key"
-	1    5000 4250
-	0    1    1    0
-$EndComp
-$Comp
-L Main_Library:R_2K_0603 R3
-U 1 1 61B509CE
-P 5150 4450
-F 0 "R3" H 5203 4496 50  0000 L CNN
-F 1 "R_2K_0603" H 5500 4550 50  0001 C CNN
-F 2 "MAIN_PCB_LIB:R_0603" H 5200 4950 50  0001 C CNN
-F 3 "" H 5150 4700 50  0001 C CNN
-F 4 "603-RT0603BRD072KL" H 5150 4950 50  0001 C CNN "Mouser"
-F 5 "2K" H 5203 4405 50  0000 L CNN "Waarde"
-	1    5150 4450
-	1    0    0    -1
-$EndComp
-Connection ~ 5150 4250
-$Comp
-L Main_Library:GND #GND05
-U 1 1 61B51C86
-P 5150 4650
-F 0 "#GND05" H 4990 4630 50  0001 C CNN
-F 1 "GND" H 4990 4630 50  0001 C CNN
-F 2 "" H 5060 4590 50  0001 C CNN
-F 3 "" H 5060 4590 50  0001 C CNN
-	1    5150 4650
-	1    0    0    -1
-$EndComp
-Text Notes 5150 4250 0    50   ~ 0
-1.5v
 $Comp
 L Main_Library:R_25K5_0603 R16
@@
 	5000 3550 5850 3550
 Connection ~ 5000 3550
+Wire Wire Line
+	5850 4250 5150 4250
+Wire Wire Line
+	5350 3950 5850 3950
+$Comp
+L Main_Library:GND #GND027
+U 1 1 61B320C3
+P 5150 4250
+F 0 "#GND027" H 4990 4230 50  0001 C CNN
+F 1 "GND" H 4990 4230 50  0001 C CNN
+F 2 "" H 5060 4190 50  0001 C CNN
+F 3 "" H 5060 4190 50  0001 C CNN
+	1    5150 4250
+	1    0    0    -1
+$EndComp
 $EndSCHEMATC
