File: versterker.kicad_pcb (KiCad board)
At the start: 2 copper layers, 65 x 56 mm, 51 parts, among them J1 J_Barreljack_3.5mm_Wurth_TH, J2 J_3.5mm_jack_SJ1-3523N, J3 40HAT, J3 J_2_screwterminal_2.54_282834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, Q1 Q_IRFZ44NPBF_N-Channel_Infine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, Q2 Q_IRFZ44NPBF_N-Channel_Infine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, U2 Val**, U3 U_LM393N_NOPB, U4 U_TC4427M_Microchip, U5 U_555_timer, U6 U_LM3914N-1_NOPB

Commit message: routed pcb
Parts:
- removed R3: R_2K_0603, MAIN_PCB_LIB:R_0603
- added C1: C_10uF_0603, MAIN_PCB_LIB:C_0603, F.Cu at (124.5, 83.2)
- added D13: D_1N4148WS_SOD323F_ONSEMI, MAIN_PCB_LIB:D_1N4148_SOD-323F_ONSEMI, F.Cu at (122.9, 94.6)
- added D14: D_1N4148WS_SOD323F_ONSEMI, MAIN_PCB_LIB:D_1N4148_SOD-323F_ONSEMI, F.Cu at (124.3, 94.7)
- added D15: D_1N4148WS_SOD323F_ONSEMI, MAIN_PCB_LIB:D_1N4148_SOD-323F_ONSEMI, F.Cu at (127.1, 103.6)
- added D16: D_1N4148WS_SOD323F_ONSEMI, MAIN_PCB_LIB:D_1N4148_SOD-323F_ONSEMI, F.Cu at (131.4, 103.6)
- added R17: R_10K_0603, MAIN_PCB_LIB:R_0603, F.Cu at (123.7, 91.7)
- R2: value R_10K_0603 -> R_1K_0603
- U2: value Val** -> U_LM358AP_TI_DIP
- moved R2 19.2 mm to (129.3, 101.7), turned to 270 degrees
- moved R5 4.54 mm to (131.3, 101.2)
- moved R4 3.43 mm to (127.2, 101.2)
- moved R18 0.23 mm to (124.5, 89.5)
Connections:
- R2 pad 1: Net-(R2-Pad1) -> Net-(D15-PadC)
- R2 pad 2: /9V -> Net-(R2-Pad2)
- R4 pad 2: Net-(R4-Pad2) -> Net-(R2-Pad2)
- R5 pad 1: Net-(R4-Pad2) -> Net-(R2-Pad2)
- R6 pad 1: Net-(R4-Pad2) -> Net-(D15-PadC)
- U6 pad 4: Net-(R2-Pad1) -> GND
- U6 pad 5: /ampsignal -> Net-(C1-Pad1)
Routing:
- net Net-(D15-PadC): track 0.00 -> 36.5 mm, vias 0 -> 2
- net Net-(R4-Pad2): track 33.7 -> 0.00 mm, vias 2 -> 0
- net /ampsignal: track 41.9 -> 24.4 mm, vias 2 -> 0
- net Net-(C1-Pad1): track 0.00 -> 15.9 mm, vias 0 -> 2
- net /Amplifier/R_channel: track 3.55 -> 7.98 mm
- net Net-(R2-Pad1): track 2.96 -> 0.00 mm
- net Net-(R2-Pad2): track 0.00 -> 2.84 mm
- net GND: track 0.00 -> 1.76 mm, vias 0 -> 144
- net /9V: track 191.1 -> 190.0 mm
- net /Amplifier/L_channel: track 8.64 -> 7.52 mm
- net Net-(D4-Pad1): track 34.6 -> 33.8 mm

Commit message: no message
Parts:
- removed R10: R_10K_0603, MAIN_PCB_LIB:R_0603
- removed R11: R_1K5_0603, MAIN_PCB_LIB:R_0603
- removed R12: R_60.4K_0603, MAIN_PCB_LIB:R_0603
- removed R16: R_25K5_0603, MAIN_PCB_LIB:R_0603
- added C8: C_680nF_TH_450V, MAIN_PCB_LIB:C_ECWFD_Panasonic, F.Cu at (95.1, 91.8)
- added C9: C_1.5uF_0603_25V, MAIN_PCB_LIB:C_0603, F.Cu at (121.6, 96.2)
- added L2: L_22uH_RFS1113_coilcraft_TH, MAIN_PCB_LIB:L_RFS1113_coilcraft, F.Cu at (86.0, 81.3)
- added R3: R_20K_0603, MAIN_PCB_LIB:R_0603, F.Cu at (111.5, 101.1)
- R5: value R_10K_0603 -> R_2K_0603
- R9: value R_20K_0603 -> R_60.4K_0603
- moved R5 19.9 mm to (112.0, 105.8), turned to 90 degrees
- moved C6 17.6 mm to (89.2, 71.2), turned to 180 degrees
- moved R4 16.0 mm to (111.5, 103.7), turned to 0 degrees
- moved J3 11.0 mm to (81.8, 91.0)
- moved D2 2.19 mm to (94.9, 106.9)
- moved R1 2.19 mm to (94.9, 109.8)
- moved R9 2.16 mm to (112.0, 99.1), turned to 270 degrees
- moved U5 1.95 mm to (106.0, 104.7)
- moved R15 1.70 mm to (95.9, 100.0)
- moved L1 1.44 mm to (99.2, 81.4)
- moved Q1 1.22 mm to (107.7, 75.9)
- moved Q2 1.22 mm to (107.5, 86.8)
- moved R7 0.29 mm to (108.7, 105.3)
- moved D14 0.25 mm to (124.6, 94.7)
- moved D13 0.25 mm to (123.1, 94.6)
Connections:
- D13 pad C: /ampsignal -> Net-(C9-Pad1)
- D14 pad A: /ampsignal -> Net-(C9-Pad1)
- J2 pad 3: /Amplifier/R_channel -> /Amplifier/L_channel
- J3 pad 2: Net-(C6-Pad1) -> Net-(C8-Pad1)
- R2 pad 2: Net-(R2-Pad2) -> /Amplifier/L_channel
- R4 pad 1: /Amplifier/R_channel -> Net-(R4-Pad1)
- R4 pad 2: Net-(R2-Pad2) -> /9V
- R5 pad 1: Net-(R2-Pad2) -> Net-(R4-Pad1)
- R5 pad 2: /Amplifier/L_channel -> GND
- R9 pad 2: Net-(C3-Pad1) -> /ampsignal
- U2 pad 3: Net-(R10-Pad1) -> Net-(R4-Pad1)
- U6 pad 6: Net-(R16-Pad1) -> Net-(R18-Pad2)
Routing:
- net /Amplifier/L_channel: track 7.52 -> 21.5 mm
- net /Amplifier/R_channel: track 7.98 -> 0.00 mm
- net /9V: track 190.0 -> 186.1 mm
- net /Triangle_wave: track 33.6 -> 37.1 mm
- net Net-(R4-Pad1): track 0.00 -> 3.35 mm
- net Net-(R10-Pad1): track 3.35 -> 0.00 mm
- net Net-(C9-Pad1): track 0.00 -> 3.22 mm
- net /ampsignal: track 24.4 -> 21.4 mm
- net Net-(R2-Pad2): track 2.84 -> 0.00 mm
- net Net-(Q1-Pad1): track 15.4 -> 12.5 mm
- net Net-(R18-Pad2): track 1.77 -> 4.37 mm
- net Net-(R16-Pad1): track 1.71 -> 0.00 mm
- net Net-(R15-Pad2): track 2.48 -> 3.14 mm
- net Net-(U5-Pad7): track 0.00 -> 0.65 mm
- net GND: track 1.76 -> 1.77 mm, vias 144 -> 126
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- added copper zone on F.Cu, net Net-(C8-Pad1)

Commit message: made gerbers
Parts:
- moved C6 0.71 mm to (88.4, 71.2)
Routing:
- net GND: vias 126 -> 119
Other:
- board text added: "+"
- board text added: "-"
- board text added: "9V"

Commit message: changed gerbers after receiving pcb
Routing:
- net Net-(C8-Pad1): vias 2 -> 0
Other:
- rule via_min_drill: 0.2 -> 0.3
