File: versterker.kicad_pcb (KiCad board)
At the start: 2 copper layers, 65 x 56 mm, 56 parts, among them J1 J_Barreljack_3.5mm_Wurth_TH, J2 J_3.5mm_jack_SJ1-3523N, J3 40HAT, J3 J_2_screwterminal_2.54_282834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, Q1 Q_IRFZ44NPBF_N-Channel_Infine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, Q2 Q_IRFZ44NPBF_N-Channel_Infine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, U2 U_LM358AP_TI_DIP, U3 U_LM393N_NOPB, U4 U_TC4427M_Microchip, U5 U_555_timer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

Commit message: changed to new kicad6
Other:
- net class Default removed
- net class default 2 removed
